File: electronic/toolman.kicad_pcb (KiCad board)
At the start: 6 copper layers, 230.1 x 95.6 mm, 257 parts, among them IC1 AT91SAM9G25-CU-999, IC2 W971GG6SB-25, IC3 NCP1529ASNT1G, IC4 CM1624-08DE, IC5 NCP1529ASNT1G, IC6 NCP1529ASNT1G, IC7 NCP1529ASNT1G, IC8 TCA8418RTWR, J1 GPIO, J10 SERIAL, J11 RJ45_Amphenol_RJMG1BD3B8K1ANR, J2 USB_OTG, J3 HISPEED, J4 USB_A, J5 USB_A, J6 Micro_SD_Card, J7 DISPLAY, J8 BACKLIGHT, J9 DEBUG, Q1 Si1442DH, SW1 CUTOFF, SW10 ZX, SW11 SELECT, SW12 ER, SW13 DF, SW14 CV, SW15 DOWN, SW16 TY, SW17 GH, SW18 BN, SW19 RIGHT, SW2 POWER, SW20 UI, SW21 JK, SW22 M., SW23 BL2, SW24 OP, SW25 L,, SW26 SPC, SW27 BL3, SW28 BKSP, SW29 ENTR, SW3 LEFT, SW30 FN, SW4 SKP, SW5 SYM, SW6 SHFT, SW7 UP, SW8 QW, SW9 AS, U1 CAT811TTBI-GT3, U2 MCP73871, U3 TPS61090, U4 KSZ8081RND, X1 ECS1612MV (50m), Y1 ABS06-127-32.768kHz, Y2 ECX33Q (12m)

Commit message: this is hard
Parts:
- removed C79: 0.1u, Capacitors_SMD:C_0402
- removed D10, D11, D12, D13, D14, D15, D16, D17, D18, D19, D20, D21, D22, D23, D24, D25, D26, D27, D28, D29, D30, D31, D4, D5, D6, D7, D8, D9: RO, Diodes_SMD:D_0603
- removed IC8: TCA8418RTWR, TCA8418RTWR:QFN50P400X400X80-25N
- removed R62: DNP, Resistors_SMD:R_0402
- removed RN1, RN2: 10k, Resistors_SMD:R_Array_Concave_4x0402
- removed SW10: ZX, Buttons_Switches_ThroughHole:SW_PUSH_6mm_h5mm
- removed SW11: SELECT, Buttons_Switches_ThroughHole:SW_PUSH_6mm_h5mm
- removed SW12: ER, Buttons_Switches_ThroughHole:SW_PUSH_6mm_h5mm
- removed SW13: DF, Buttons_Switches_ThroughHole:SW_PUSH_6mm_h5mm
- removed SW14: CV, Buttons_Switches_ThroughHole:SW_PUSH_6mm_h5mm
- removed SW15: DOWN, Buttons_Switches_ThroughHole:SW_PUSH_6mm_h5mm
- removed SW16: TY, Buttons_Switches_ThroughHole:SW_PUSH_6mm_h5mm
- removed SW17: GH, Buttons_Switches_ThroughHole:SW_PUSH_6mm_h5mm
- removed SW18: BN, Buttons_Switches_ThroughHole:SW_PUSH_6mm_h5mm
- removed SW19: RIGHT, Buttons_Switches_ThroughHole:SW_PUSH_6mm_h5mm
- removed SW20: UI, Buttons_Switches_ThroughHole:SW_PUSH_6mm_h5mm
- removed SW21: JK, Buttons_Switches_ThroughHole:SW_PUSH_6mm_h5mm
- removed SW22: M., Buttons_Switches_ThroughHole:SW_PUSH_6mm_h5mm
- removed SW23: BL2, Buttons_Switches_ThroughHole:SW_PUSH_6mm_h5mm
- removed SW24: OP, Buttons_Switches_ThroughHole:SW_PUSH_6mm_h5mm
- removed SW25: L,, Buttons_Switches_ThroughHole:SW_PUSH_6mm_h5mm
- removed SW26: SPC, Buttons_Switches_ThroughHole:SW_PUSH_6mm_h5mm
- removed SW27: BL3, Buttons_Switches_ThroughHole:SW_PUSH_6mm_h5mm
- removed SW28: BKSP, Buttons_Switches_ThroughHole:SW_PUSH_6mm_h5mm
- removed SW29: ENTR, Buttons_Switches_ThroughHole:SW_PUSH_6mm_h5mm
- removed SW3: LEFT, Buttons_Switches_ThroughHole:SW_PUSH_6mm_h5mm
- removed SW30: FN, Buttons_Switches_ThroughHole:SW_PUSH_6mm_h5mm
- removed SW4: SKP, Buttons_Switches_ThroughHole:SW_PUSH_6mm_h5mm
- removed SW5: SYM, Buttons_Switches_ThroughHole:SW_PUSH_6mm_h5mm
- removed SW6: SHFT, Buttons_Switches_ThroughHole:SW_PUSH_6mm_h5mm
- removed SW7: UP, Buttons_Switches_ThroughHole:SW_PUSH_6mm_h5mm
- removed SW8: QW, Buttons_Switches_ThroughHole:SW_PUSH_6mm_h5mm
- removed SW9: AS, Buttons_Switches_ThroughHole:SW_PUSH_6mm_h5mm
- added J12: KEYBOARD, Pin_Headers:Pin_Header_Angled_1x06_Pitch1.27mm, F.Cu at (167.7, 132.2)
- moved IC2 0.25 mm to (84.2, 46.5)
Routing:
- net /D8: track 30.1 -> 0.00 mm, vias 2 -> 0
- net /SDCKE: track 25.6 -> 0.00 mm, vias 3 -> 0
- net /D4: track 25.3 -> 0.00 mm, vias 3 -> 0
- net /RASn: track 25.1 -> 0.00 mm, vias 2 -> 0
- net /D3: track 25.1 -> 0.00 mm, vias 2 -> 0
- net /DQS1: track 25.0 -> 0.00 mm, vias 2 -> 0
- net /CASn: track 25.0 -> 0.00 mm, vias 2 -> 0
- net /D12: track 25.0 -> 0.00 mm, vias 2 -> 0
- net /A10: track 25.0 -> 0.00 mm, vias 2 -> 0
- net /D5: track 25.0 -> 0.00 mm, vias 2 -> 0
- net /A13: track 25.0 -> 0.00 mm, vias 2 -> 0
- net /D13: track 25.0 -> 0.00 mm, vias 2 -> 0
- net /A6: track 25.0 -> 0.00 mm, vias 2 -> 0
- net /D7: track 25.0 -> 0.00 mm, vias 2 -> 0
- net /D14: track 25.0 -> 0.00 mm, vias 2 -> 0
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Other:
- net class DDR_ACB added: clearance 0.127, trace_width 0.0889, via_dia 0.45, via_drill 0.2
- net class DDR_DB added: clearance 0.127, trace_width 0.0889, via_dia 0.45, via_drill 0.2
