File: electronic/toolman.sch (KiCad schematic (older format))
At the start: 150 parts

Commit message: bee gee aay
Parts:
- added C65, C67, C69, C70: 1u, Capacitors_SMD:C_0402, symbol Device:C
- added C71, C74, C77, C78, C79: 0.1u, Capacitors_SMD:C_0402, symbol Device:C
- added C73, C75, C76: 2.2u, Capacitors_SMD:C_0402, symbol Device:C
- added D10, D11, D12, D13, D14, D15, D16, D17, D18, D19, D20, D21, D22, D23, D24, D25, D26, D27, D28, D29, D30, D31, D4, D5, D6, D7, D8, D9: RO, Diodes_SMD:D_0603, symbol Device:D_Small
- added FB1: Ferrite, w_smd_inductors:inductor_smd_0603, symbol Device:Ferrite_Bead_Small
- added IC8: TCA8418RTWR, TCA8418RTWR:QFN50P400X400X80-25N, symbol TCA8418RTWR:TCA8418RTWR
- added J1: GPIO, Pin_Headers:Pin_Header_Straight_2x20_Pitch1.27mm, symbol Connector_Generic:Conn_02x20_Odd_Even
- added J10: SERIAL, Pin_Headers:Pin_Header_Angled_1x04_Pitch2.54mm, symbol Connector_Generic:Conn_01x04
- added J11: RJ45_Amphenol_RJMG1BD3B8K1ANR, w_conn_pc:rj45-wiznet-rb1-125bag1a, symbol Connector:RJ45_Amphenol_RJMG1BD3B8K1ANR
- added J3: HISPEED, Pin_Headers:Pin_Header_Straight_2x14_Pitch1.27mm, symbol Connector_Generic:Conn_02x14_Odd_Even
- added J7: DISPLAY, ER-CON25HB:ER-CON25HB, symbol Connector_Generic:Conn_01x25
- added J8: BACKLIGHT, 1769:1769, symbol Connector_Generic:Conn_01x02
- added J9: DEBUG, Pin_Headers:Pin_Header_Straight_2x09_Pitch1.27mm, symbol Connector_Generic:Conn_02x09_Odd_Even
- added L13: 10u, w_smd_inductors:inductor_smd_0603, symbol Device:L
- added Q1: Si1442DH, TO_SOT_Packages_SMD:SOT-363_SC-70-6, symbol Transistor_FET:Si1442DH
- added R23, R50, R53, R57, R59, R62: DNP, Resistors_SMD:R_0402, symbol Device:R
- added R51, R52, R56, R58: 1k, Resistors_SMD:R_0402, symbol Device:R
- added R54: 6.49k, Resistors_SMD:R_0402, symbol Device:R
- added R55: 10k, Resistors_SMD:R_0402, symbol Device:R
- added R60, R61: 47k, Resistors_SMD:R_0402, symbol Device:R
- added RN1, RN2: 10k, Resistors_SMD:R_Array_Concave_4x0402, symbol Device:R_Pack04
- added SW1: CUTOFF, Buttons_Switches_SMD:SW_DIP_x1_W5.08mm_Slide_Copal_CHS-A, symbol Switch:SW_DIP_x01
- added SW10: ZX, Buttons_Switches_ThroughHole:SW_PUSH_6mm_h5mm, symbol Switch:SW_Push_45deg
- added SW11: SELECT, Buttons_Switches_ThroughHole:SW_PUSH_6mm_h5mm, symbol Switch:SW_Push_45deg
- added SW12: ER, Buttons_Switches_ThroughHole:SW_PUSH_6mm_h5mm, symbol Switch:SW_Push_45deg
- added SW13: DF, Buttons_Switches_ThroughHole:SW_PUSH_6mm_h5mm, symbol Switch:SW_Push_45deg
- added SW14: CV, Buttons_Switches_ThroughHole:SW_PUSH_6mm_h5mm, symbol Switch:SW_Push_45deg
- added SW15: DOWN, Buttons_Switches_ThroughHole:SW_PUSH_6mm_h5mm, symbol Switch:SW_Push_45deg
- added SW16: TY, Buttons_Switches_ThroughHole:SW_PUSH_6mm_h5mm, symbol Switch:SW_Push_45deg
- added SW17: GH, Buttons_Switches_ThroughHole:SW_PUSH_6mm_h5mm, symbol Switch:SW_Push_45deg
- added SW18: BN, Buttons_Switches_ThroughHole:SW_PUSH_6mm_h5mm, symbol Switch:SW_Push_45deg
- added SW19: RIGHT, Buttons_Switches_ThroughHole:SW_PUSH_6mm_h5mm, symbol Switch:SW_Push_45deg
- added SW2: POWER, Buttons_Switches_SMD:Panasonic_EVQPUL_EVQPUC, symbol Switch:SW_Push_45deg
- added SW20: UI, Buttons_Switches_ThroughHole:SW_PUSH_6mm_h5mm, symbol Switch:SW_Push_45deg
- added SW21: JK, Buttons_Switches_ThroughHole:SW_PUSH_6mm_h5mm, symbol Switch:SW_Push_45deg
- added SW22: M., Buttons_Switches_ThroughHole:SW_PUSH_6mm_h5mm, symbol Switch:SW_Push_45deg
- added SW23: BL2, Buttons_Switches_ThroughHole:SW_PUSH_6mm_h5mm, symbol Switch:SW_Push_45deg
- added SW24: OP, Buttons_Switches_ThroughHole:SW_PUSH_6mm_h5mm, symbol Switch:SW_Push_45deg
- added SW25: L,, Buttons_Switches_ThroughHole:SW_PUSH_6mm_h5mm, symbol Switch:SW_Push_45deg
- added SW26: SPC, Buttons_Switches_ThroughHole:SW_PUSH_6mm_h5mm, symbol Switch:SW_Push_45deg
- added SW27: BL3, Buttons_Switches_ThroughHole:SW_PUSH_6mm_h5mm, symbol Switch:SW_Push_45deg
- added SW28: BKSP, Buttons_Switches_ThroughHole:SW_PUSH_6mm_h5mm, symbol Switch:SW_Push_45deg
- added SW29: ENTR, Buttons_Switches_ThroughHole:SW_PUSH_6mm_h5mm, symbol Switch:SW_Push_45deg
- added SW3: LEFT, Buttons_Switches_ThroughHole:SW_PUSH_6mm_h5mm, symbol Switch:SW_Push_45deg
- added SW30: FN, Buttons_Switches_ThroughHole:SW_PUSH_6mm_h5mm, symbol Switch:SW_Push_45deg
- added SW4: SKP, Buttons_Switches_ThroughHole:SW_PUSH_6mm_h5mm, symbol Switch:SW_Push_45deg
- added SW5: SYM, Buttons_Switches_ThroughHole:SW_PUSH_6mm_h5mm, symbol Switch:SW_Push_45deg
- added SW6: SHFT, Buttons_Switches_ThroughHole:SW_PUSH_6mm_h5mm, symbol Switch:SW_Push_45deg
- added SW7: UP, Buttons_Switches_ThroughHole:SW_PUSH_6mm_h5mm, symbol Switch:SW_Push_45deg
- added SW8: QW, Buttons_Switches_ThroughHole:SW_PUSH_6mm_h5mm, symbol Switch:SW_Push_45deg
- added SW9: AS, Buttons_Switches_ThroughHole:SW_PUSH_6mm_h5mm, symbol Switch:SW_Push_45deg
- added TP1: TEST_Vcharge, Measurement_Points:Measurement_Point_Round-SMD-Pad_Small, symbol Connector:TestPoint
- added TP2: TEST_Vbatt, Measurement_Points:Measurement_Point_Round-SMD-Pad_Small, symbol Connector:TestPoint
- added TP3: TEST_1.8v, Measurement_Points:Measurement_Point_Round-SMD-Pad_Small, symbol Connector:TestPoint
- added TP4: TEST_5v, Measurement_Points:Measurement_Point_Round-SMD-Pad_Small, symbol Connector:TestPoint
- added TP5: TEST_1.0v, Measurement_Points:Measurement_Point_Round-SMD-Pad_Small, symbol Connector:TestPoint
- added TP6: TEST_3.3v, Measurement_Points:Measurement_Point_Round-SMD-Pad_Small, symbol Connector:TestPoint
- added TP7: TEST_Vbackup, Measurement_Points:Measurement_Point_Round-SMD-Pad_Small, symbol Connector:TestPoint
- added TP8: TEST_1.2v, Measurement_Points:Measurement_Point_Round-SMD-Pad_Small, symbol Connector:TestPoint
- added TP9: TEST_LED, Measurement_Points:Measurement_Point_Round-SMD-Pad_Small, symbol Connector:TestPoint
- added X1: ECS1612MV (50m), ECS-1612MV-250-CN-TR:ECS1612MV250CNTR, symbol Oscillator:XO32
- BT1: renamed from BT?; footprint (none) -> 1769:1769
- C1, C10, C11, C12, C13, C14, C15, C16, C17, C18, C19, C2, C20, C21, C22, C23, C24, C25, C26, C27, C28, C29, C3, C30, C31, C32, C33, C34, C35, C36, C37, C38, C39, C4, C40, C41, C42, C43, C44, C45, C46, C47, C48, C49, C5, C50, C51, C52, C54, C55, C56, C57, C58, C59, C6, C60, C62, C64, C7, C8, C9: renamed from C?; footprint (none) -> Capacitors_SMD:C_0402
- C53: renamed from C?; footprint (none) -> Capacitors_SMD:CP_Elec_6.3x5.3
- C61, C63, C66, C68: renamed from C?; footprint (none) -> Capacitors_SMD:C_0603
- D1, D2, D3: renamed from D?; footprint (none) -> LEDs:LED_0805
- FL1, FL2, FL3: renamed from FL?; footprint (none) -> DLP11SA900HL2L:DLP11S
- IC1: renamed from IC?; footprint BGA217C80P17X17_1500X1500X140 -> AT91SAM9G25-CU-999:BGA217C80P17X17_1500X1500X140
- IC2: renamed from IC?; footprint BGA84C80P9X15_800X1250X120 -> W971GG6SB-25:BGA84C80P9X15_800X1250X120
- IC3, IC5, IC6, IC7: renamed from IC?; footprint SOT95P275X110-5N -> NCP1529ASNT1G:SOT95P275X110-5N
- IC4: renamed from IC?; footprint SON40P135X330X55-17N -> CM1624-08DE:SON40P135X330X55-17N
- J2: renamed from J?; footprint (none) -> Connect:USB_Micro-B_10103594-0001LF
- J4, J5: renamed from J?; footprint (none) -> w_conn_pc:conn_usb_A
- J6: renamed from J?; footprint (none) -> 1051620001:1051620001
- L1, L12, L2, L4, L5, L6, L8, L9: renamed from L?; footprint (none) -> w_smd_inductors:inductor_smd_0603
- L10, L11, L3, L7: renamed from L?; footprint (none) -> w_smd_inductors:inductor_smd_0805
- R1, R10, R11, R12, R13, R14, R15, R16, R17, R18, R19, R2, R20, R21, R22, R24, R25, R26, R27, R28, R29, R3, R31, R32, R34, R35, R36, R37, R38, R39, R4, R40, R41, R42, R43, R44, R45, R46, R47, R48, R49, R5, R6, R7, R8, R9: renamed from R?; footprint (none) -> Resistors_SMD:R_0402
- R30: renamed from R?; value R -> 1k; footprint (none) -> Resistors_SMD:R_0402
- R33: renamed from R?; value R -> 1.4k; footprint (none) -> Resistors_SMD:R_0402
- U1: renamed from U?; footprint Package_TO_SOT_SMD:SOT-143 -> CAT811STBI-GT3:4-PIN-SOT-143(BI-SUFFIX-CASE-527AF)
- U2: renamed from U?; footprint Package_DFN_QFN:QFN-20-1EP_4x4mm_P0.5mm_EP2.5x2.5mm -> Housings_DFN_QFN:QFN-20-1EP_4x4mm_Pitch0.5mm
- U3: renamed from U?; footprint Package_DFN_QFN:Texas_S-PVQFN-N16_EP2.7x2.7mm_ThermalVias -> TPS61090RSAR:QFN65P400X400X100-17N
- U4: renamed from U?; value KSZ8081RNA -> KSZ8081RND; footprint Package_DFN_QFN:QFN-24-1EP_4x4mm_P0.5mm_EP2.6x2.6mm -> Housings_DFN_QFN:QFN-24-1EP_4x4mm_Pitch0.5mm
- Y1: renamed from Y?; value 32.768k -> ABS06-127-32.768kHz; footprint (none) -> Crystals:Crystal_SMD_TXC_9HT11-2pin_2.0x1.2mm_HandSoldering
- Y2: renamed from Y?; value 12m -> ECX33Q (12m); footprint (none) -> Crystals:Crystal_SMD_EuroQuartz_MT-4pin_3.2x2.5mm
Connections:
- net +1V0: now also TP5.1
- net +1V8: now also R23.2, TP3.1
- net +3V3: now also U4.14 (VDDIO), C71.2, C75.1, C77.1, C79.1, FB1.1, IC8.21 (VCC), J1.1 (Pin_1), J11.R4 (TCT), J11.R5 (RCT), J3.1 (Pin_1), J3.28 (Pin_28), J7.11 (Pin_11), J7.12 (Pin_12), J7.14 (Pin_14), J7.23 (Pin_23), J7.6 (Pin_6), J8.1 (Pin_1), J9.4 (Pin_4), R51.1, R52.1, R56.1, R57.1, R57.2, R58.1, R59.1, R60.1, R61.1, RN1.5 (R4.2), RN1.6 (R3.2), RN1.7 (R2.2), RN1.8 (R1.2), RN2.5 (R4.2), RN2.6 (R3.2), RN2.7 (R2.2), RN2.8 (R1.2), TP6.1, X1.1 (EN), X1.4 (V+)
- net +5V: now also J1.2 (Pin_2), TP4.1
- net +BATT: now also TP2.1
- net BATTVOLT: now also IC1.B1 (PB17)
- net BMS: now also J9.13 (Pin_13)
- net CHARGED: now also IC1.F4 (PC1)
- net CHARGING: now also IC1.E2 (PC0)
- net CPU_NRST: now also U4.24 (~RST), IC8.20 (~RESET), J10.2 (Pin_2), J9.15 (Pin_15), R53.1, R53.2, R62.1, R62.2
- net CPU_NTRST: now also J9.16 (Pin_16)
- net CPU_SHDN: now also U3.11 (EN), J9.18 (Pin_18)
- net CPU_WKUP: now also J9.14 (Pin_14), R55.1, SW2.1
- net GND: now also U4.22 (GND), U4.25 (GND), C65.2, C69.2, C70.2, C71.1, C73.2, C74.2, C75.2, C76.1, C77.2, C78.1, C79.2, IC8.19 (GND), IC8.25 (EP), J1.19 (Pin_19), J1.23 (Pin_23), J1.27 (Pin_27), J1.33 (Pin_33), J1.34 (Pin_34), J1.37 (Pin_37), J10.1 (Pin_1), J11.R8 (GND), J3.10 (Pin_10), J3.11 (Pin_11), J3.14 (Pin_14), J3.15 (Pin_15), J3.18 (Pin_18), J3.19 (Pin_19), J3.2 (Pin_2), J3.22 (Pin_22), J3.23 (Pin_23), J3.26 (Pin_26), J3.27 (Pin_27), J3.3 (Pin_3), J3.6 (Pin_6), J3.7 (Pin_7), J7.1 (Pin_1), J7.10 (Pin_10), J7.25 (Pin_25), J7.7 (Pin_7), J9.10 (Pin_10), J9.2 (Pin_2), L13.1, Q1.4 (S), R23.1, R54.1, R59.2, SW2.2, X1.2 (GND)
- net JTAGSEL: now also J9.11 (Pin_11)
- net LOWBATTERY: now also IC1.F3 (PC2)
- net RTCK: now also J9.12 (Pin_12)
- net TCK: now also J9.1 (Pin_1)
- net TDI: now also J9.9 (Pin_9)
- net TDO: now also J9.3 (Pin_3)
- net TMS: now also J9.5 (Pin_5)
- net VEE: now also J1.17 (Pin_17), R55.2, TP7.1
- net VPP: now also SW1.2; no longer U2.1 (OUT), U2.20 (OUT)
- net PB16_AD5: now reaches IC1.A1 (PB16)
- net PB16_AD5: now also J1.28 (Pin_28)
- net PB13_DISPLAY_BACKLIGHT: now reaches IC1.A2 (PB13)
- net PB13_DISPLAY_BACKLIGHT: now also Q1.3 (G)
- net PB10_ETX1: now reaches IC1.B2 (PB10)
- net PB10_ETX1: now also U4.21 (TXD1)
- net PB12_DISPLAY_RESET: now reaches IC1.B4 (PB12)
- net PB12_DISPLAY_RESET: now also J7.13 (Pin_13)
- net PB9_ETX0: now reaches IC1.C1 (PB9)
- net PB9_ETX0: now also U4.20 (TXD0)
- net PB7_ETXEN: now reaches IC1.C2 (PB7)
- net PB7_ETXEN: now also U4.19 (TXEN)
- net PB15_AD4: now reaches IC1.C3 (PB15)
- net PB15_AD4: now also J1.20 (Pin_20)
- net PB14_DISPLAY_ADDRESS: now reaches IC1.C4 (PB14)
- net PB14_DISPLAY_ADDRESS: now also J7.21 (Pin_21)
- net PB4_ETXCK: now reaches IC1.D1 (PB4)
- net PB4_ETXCK: now also U4.16 (REF_CLK), R50.1, R50.2
- net PB2_ERXER: now reaches IC1.D2 (PB2)
- net PB2_ERXER: now also U4.17 (RXER)
- net PB0_ERX0: now reaches IC1.D3 (PB0)
- net PB0_ERX0: now also U4.13 (RXD0)
- net PB1_ERX1: now reaches IC1.D4 (PB1)
- net PB1_ERX1: now also U4.12 (RXD1)
- net PC4: now reaches IC1.E1 (PC4)
- net PC4: now also J1.5 (Pin_5)
- net PB3_ERXDV: now reaches IC1.E4 (PB3)
- net PB3_ERXDV: now also U4.15 (CRS_DV/PHYAD[1:0])
- net PC7: now reaches IC1.F1 (PC7)
- net PC7: now also J1.11 (Pin_11)
- net PC6: now reaches IC1.F2 (PC6)
- net PC6: now also J1.9 (Pin_9)
- net PC8: now reaches IC1.G1 (PC8)
- net PC8: now also J1.13 (Pin_13)
- net PC10: now reaches IC1.G2 (PC10)
- net PC10: now also J1.4 (Pin_4)
- net PC9: now reaches IC1.G3 (PC9)
- net PC9: now also J1.15 (Pin_15)
- net PC5: now reaches IC1.G4 (PC5)
- net PC5: now also J1.7 (Pin_7)
- net PC14: now reaches IC1.H1 (PC14)
- net PC14: now also J1.12 (Pin_12)
- net PC3: now reaches IC1.H2 (PC3)
- net PC3: now also J1.3 (Pin_3)
- net PC11: now reaches IC1.H3 (PC11)
- net PC11: now also J1.6 (Pin_6)
- net PC16: now reaches IC1.J1 (PC16)
- net PC16: now also J1.16 (Pin_16)
- net PC15: now reaches IC1.J2 (PC15)
- net PC15: now also J1.14 (Pin_14)
- net PC12: now reaches IC1.J3 (PC12)
- net PC12: now also J1.8 (Pin_8)
- net PC23_RXD3: now reaches IC1.J4 (PC23)
- net PC23_RXD3: now also J1.39 (Pin_39)
- net PC20_PWM2: now reaches IC1.K1 (PC20)
- net PC20_PWM2: now also J3.20 (Pin_20)
- net PC18_PWM0: now reaches IC1.K2 (PC18)
- net PC18_PWM0: now also J3.21 (Pin_21)
- net PC24_RTS3: now reaches IC1.K3 (PC24)
- net PC24_RTS3: now also J1.36 (Pin_36)
- net PC17: now reaches IC1.L1 (PC17)
- net PC17: now also J1.18 (Pin_18)
- net PC13: now reaches IC1.L2 (PC13)
- net PC13: now also J1.10 (Pin_10)
- net PA0_TXD0: now reaches IC1.L3 (PA0)
- net PA0_TXD0: now also J1.21 (Pin_21)
- net PA2_RTS0: now reaches IC1.L4 (PA2)
- net PA2_RTS0: now also J1.22 (Pin_22)
- net PC25_CTS3: now reaches IC1.M2 (PC25)
- net PC25_CTS3: now also J1.38 (Pin_38)
- net PC21_PWM3: now reaches IC1.M3 (PC21)
- net PC21_PWM3: now also J3.24 (Pin_24)
- net PC19_PWM1: now reaches IC1.N3 (PC19)
- net PC19_PWM1: now also J3.25 (Pin_25)
- net PA3_CTS0: now reaches IC1.N4 (PA3)
- net PA3_CTS0: now also J1.24 (Pin_24)
- net PA1_RXD0: now reaches IC1.P1 (PA1)
- net PA1_RXD0: now also J1.25 (Pin_25)
- net PC26_SCK3: now reaches IC1.P2 (PC26)
- net PC26_SCK3: now also J1.40 (Pin_40)
- net PC22_TXD3: now reaches IC1.P3 (PC22)
- net PC22_TXD3: now also J1.35 (Pin_35)
- net PA8_RXD2: now reaches IC1.P4 (PA8)
- net PA8_RXD2: now also J1.32 (Pin_32)
- net PA27_TIOB0: now reaches IC1.P8 (PA27)
- net PA27_TIOB0: now also J3.5 (Pin_5)
- net PA5_TXD1: now reaches IC1.R1 (PA5)
- net PA5_TXD1: now also J1.29 (Pin_29)
- net PA7_TXD2: now reaches IC1.R3 (PA7)
- net PA7_TXD2: now also J1.30 (Pin_30)
- net PA6_RXD1: now reaches IC1.R4 (PA6)
- net PA6_RXD1: now also J1.31 (Pin_31)
- net PA22_TIOA1: now reaches IC1.R6 (PA22)
- net PA22_TIOA1: now also J3.13 (Pin_13)
- net PA26_TCLK2: now reaches IC1.R7 (PA26)
- net PA26_TCLK2: now also J3.16 (Pin_16)
- net PA30_TWD0: now reaches IC1.R8 (PA30)
- net PA30_TWD0: now also IC8.22 (SDA), R60.2
- net PA29_KEY_INT: now reaches IC1.R9 (PA29)
- net PA29_KEY_INT: now also IC8.24 (~INT)
- net PA10_DTXD: now reaches IC1.T1 (PA10)
- net PA10_DTXD: now also J10.4 (Pin_4)
- net PA12_SPI0_MOSI: now reaches IC1.T2 (PA12)
- net PA12_SPI0_MOSI: now also J7.22 (Pin_22)
- net PA4_SCK0: now reaches IC1.T3 (PA4)
- net PA4_SCK0: now also J1.26 (Pin_26)
- net PA13_SPI0_SPCK: now reaches IC1.T4 (PA13)
- net PA13_SPI0_SPCK: now also J7.24 (Pin_24)
- net PA21_TIOA0: now reaches IC1.T6 (PA21)
- net PA21_TIOA0: now also J3.9 (Pin_9)
- net PA24_TCLK0: now reaches IC1.T7 (PA24)
- net PA24_TCLK0: now also J3.8 (Pin_8)
- net PA25_TCLK1: now reaches IC1.T8 (PA25)
- net PA25_TCLK1: now also J3.12 (Pin_12)
- net PA14_SPI0_NPCS0: now reaches IC1.U2 (PA14)
- net PA14_SPI0_NPCS0: now also J7.9 (Pin_9)
- net PA9_DRDX: now reaches IC1.U3 (PA9)
- net PA9_DRDX: now also J10.3 (Pin_3)
- net PA23_TIOA2: now reaches IC1.U7 (PA23)
- net PA23_TIOA2: now also J3.17 (Pin_17)
- net PA28_TIOB1: now reaches IC1.U8 (PA28)
- net PA28_TIOB1: now also J3.4 (Pin_4)
- net PA31_TWCK0: now reaches IC1.U9 (PA31)
- net PA31_TWCK0: now also IC8.23 (SCL), R61.2
- net at J5.5 (Shield): now also L11.2
- net at U4.1 (VDD_1.2): now also C73.1, C74.1, TP8.1
- net at U4.10 (MDIO): now also R51.2
- net at U4.18 (INTRP): now also R52.2
- net at U4.2 (VDDA_3.3): now also C76.2, C78.2, FB1.2
- net at U4.23 (LED0/ANEN_SPEED): now also J11.L3 (LEDG_K)
- net at U4.3 (RXM): now also J11.R6 (RD-)
- net at U4.4 (RXP): now also J11.R3 (RD+)
- net at U4.5 (TXM): now also J11.R2 (TD-)
- net at U4.6 (TXP): now also J11.R1 (TD+)
- net at U4.8 (XI): now also X1.3 (OUT)
- net at U4.9 (REXT): now also R54.2
- net DDR_CLK renamed DDR_CLK_P
- net DDR_CLKn renamed DDR_CLK_N
- new net: J11.13 (SHIELD), L13.2
- new net: J11.L1 (LEDY_A), R58.2
- new net: J11.L2 (LEDY_K), TP9.1
- new net: J11.L4 (LEDG_A), R56.2
- new net: SW1.1, TP1.1, U2.1 (OUT), U2.20 (OUT)
- new net: C69.1, J7.2 (Pin_2)
- new net: C67.2, J7.3 (Pin_3)
- new net: C67.1, J7.4 (Pin_4)
- new net: C70.1, J7.5 (Pin_5)
- new net: C65.1, J7.8 (Pin_8)
- new net: J8.2 (Pin_2), Q1.1 (D), Q1.2 (D), Q1.5 (D), Q1.6 (D)
- new net: IC8.2 (ROW6), SW3.1, SW4.1, SW5.1, SW6.1
- new net: D4.2 (A), SW3.2
- new net: IC8.3 (ROW5), SW10.1, SW7.1, SW8.1, SW9.1
- new net: D8.2 (A), SW7.2
- new net: IC8.4 (ROW4), SW11.1, SW12.1, SW13.1, SW14.1
- new net: D12.2 (A), SW11.2
- new net: IC8.5 (ROW3), SW15.1, SW16.1, SW17.1, SW18.1
- new net: D16.2 (A), SW15.2
- new net: IC8.6 (ROW2), SW19.1, SW20.1, SW21.1, SW22.1
- new net: D20.2 (A), SW19.2
- new net: IC8.7 (ROW1), SW23.1, SW24.1, SW25.1, SW26.1
- new net: D24.2 (A), SW23.2
- new net: IC8.8 (ROW0), SW27.1, SW28.1, SW29.1, SW30.1
- new net: D28.2 (A), SW27.2
- new net: D12.1 (K), D16.1 (K), D20.1 (K), D24.1 (K), D28.1 (K), D4.1 (K), D8.1 (K), IC8.9 (COL0)
- new net: D5.2 (A), SW4.2
- new net: D9.2 (A), SW8.2
- new net: D13.2 (A), SW12.2
- new net: D17.2 (A), SW16.2
- new net: D21.2 (A), SW20.2
- new net: D25.2 (A), SW24.2
- new net: D29.2 (A), SW28.2
- new net: D13.1 (K), D17.1 (K), D21.1 (K), D25.1 (K), D29.1 (K), D5.1 (K), D9.1 (K), IC8.10 (COL1)
- new net: D6.2 (A), SW5.2
- new net: D10.2 (A), SW9.2
- new net: D14.2 (A), SW13.2
- new net: D18.2 (A), SW17.2
- new net: D22.2 (A), SW21.2
- new net: D26.2 (A), SW25.2
- new net: D30.2 (A), SW29.2
- new net: D10.1 (K), D14.1 (K), D18.1 (K), D22.1 (K), D26.1 (K), D30.1 (K), D6.1 (K), IC8.11 (COL2)
- new net: D7.2 (A), SW6.2
- new net: D11.2 (A), SW10.2
- new net: D15.2 (A), SW14.2
- new net: D19.2 (A), SW18.2
- new net: D23.2 (A), SW22.2
- new net: D27.2 (A), SW26.2
- new net: D31.2 (A), SW30.2
- new net: D11.1 (K), D15.1 (K), D19.1 (K), D23.1 (K), D27.1 (K), D31.1 (K), D7.1 (K), IC8.12 (COL3)
- new net: IC8.1 (ROW7), RN2.3 (R3.1)
- new net: IC8.13 (COL4), RN2.2 (R2.1)
- new net: IC8.14 (COL5), RN2.1 (R1.1)
- new net: IC8.15 (COL6), RN1.4 (R4.1)
- new net: IC8.16 (COL7), RN1.3 (R3.1)
- new net: IC8.17 (COL8), RN1.2 (R2.1)
- new net: IC8.18 (COL9), RN1.1 (R1.1)
- no-connect marks 16 -> 69
Other:
- moved on the sheet: C27, C28, C29, C30, C31, C32, C33, C34, C35, C36, C38, C39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

Commit message: this is hard
Parts:
- removed C79: 0.1u, Capacitors_SMD:C_0402, symbol Device:C
- removed D10, D11, D12, D13, D14, D15, D16, D17, D18, D19, D20, D21, D22, D23, D24, D25, D26, D27, D28, D29, D30, D31, D4, D5, D6, D7, D8, D9: RO, Diodes_SMD:D_0603, symbol Device:D_Small
- removed IC8: TCA8418RTWR, TCA8418RTWR:QFN50P400X400X80-25N, symbol TCA8418RTWR:TCA8418RTWR
- removed R62: DNP, Resistors_SMD:R_0402, symbol Device:R
- removed RN1, RN2: 10k, Resistors_SMD:R_Array_Concave_4x0402, symbol Device:R_Pack04
- removed SW10: ZX, Buttons_Switches_ThroughHole:SW_PUSH_6mm_h5mm, symbol Switch:SW_Push_45deg
- removed SW11: SELECT, Buttons_Switches_ThroughHole:SW_PUSH_6mm_h5mm, symbol Switch:SW_Push_45deg
- removed SW12: ER, Buttons_Switches_ThroughHole:SW_PUSH_6mm_h5mm, symbol Switch:SW_Push_45deg
- removed SW13: DF, Buttons_Switches_ThroughHole:SW_PUSH_6mm_h5mm, symbol Switch:SW_Push_45deg
- removed SW14: CV, Buttons_Switches_ThroughHole:SW_PUSH_6mm_h5mm, symbol Switch:SW_Push_45deg
- removed SW15: DOWN, Buttons_Switches_ThroughHole:SW_PUSH_6mm_h5mm, symbol Switch:SW_Push_45deg
- removed SW16: TY, Buttons_Switches_ThroughHole:SW_PUSH_6mm_h5mm, symbol Switch:SW_Push_45deg
- removed SW17: GH, Buttons_Switches_ThroughHole:SW_PUSH_6mm_h5mm, symbol Switch:SW_Push_45deg
- removed SW18: BN, Buttons_Switches_ThroughHole:SW_PUSH_6mm_h5mm, symbol Switch:SW_Push_45deg
- removed SW19: RIGHT, Buttons_Switches_ThroughHole:SW_PUSH_6mm_h5mm, symbol Switch:SW_Push_45deg
- removed SW20: UI, Buttons_Switches_ThroughHole:SW_PUSH_6mm_h5mm, symbol Switch:SW_Push_45deg
- removed SW21: JK, Buttons_Switches_ThroughHole:SW_PUSH_6mm_h5mm, symbol Switch:SW_Push_45deg
- removed SW22: M., Buttons_Switches_ThroughHole:SW_PUSH_6mm_h5mm, symbol Switch:SW_Push_45deg
- removed SW23: BL2, Buttons_Switches_ThroughHole:SW_PUSH_6mm_h5mm, symbol Switch:SW_Push_45deg
- removed SW24: OP, Buttons_Switches_ThroughHole:SW_PUSH_6mm_h5mm, symbol Switch:SW_Push_45deg
- removed SW25: L,, Buttons_Switches_ThroughHole:SW_PUSH_6mm_h5mm, symbol Switch:SW_Push_45deg
- removed SW26: SPC, Buttons_Switches_ThroughHole:SW_PUSH_6mm_h5mm, symbol Switch:SW_Push_45deg
- removed SW27: BL3, Buttons_Switches_ThroughHole:SW_PUSH_6mm_h5mm, symbol Switch:SW_Push_45deg
- removed SW28: BKSP, Buttons_Switches_ThroughHole:SW_PUSH_6mm_h5mm, symbol Switch:SW_Push_45deg
- removed SW29: ENTR, Buttons_Switches_ThroughHole:SW_PUSH_6mm_h5mm, symbol Switch:SW_Push_45deg
- removed SW3: LEFT, Buttons_Switches_ThroughHole:SW_PUSH_6mm_h5mm, symbol Switch:SW_Push_45deg
- removed SW30: FN, Buttons_Switches_ThroughHole:SW_PUSH_6mm_h5mm, symbol Switch:SW_Push_45deg
- removed SW4: SKP, Buttons_Switches_ThroughHole:SW_PUSH_6mm_h5mm, symbol Switch:SW_Push_45deg
- removed SW5: SYM, Buttons_Switches_ThroughHole:SW_PUSH_6mm_h5mm, symbol Switch:SW_Push_45deg
- removed SW6: SHFT, Buttons_Switches_ThroughHole:SW_PUSH_6mm_h5mm, symbol Switch:SW_Push_45deg
- removed SW7: UP, Buttons_Switches_ThroughHole:SW_PUSH_6mm_h5mm, symbol Switch:SW_Push_45deg
- removed SW8: QW, Buttons_Switches_ThroughHole:SW_PUSH_6mm_h5mm, symbol Switch:SW_Push_45deg
- removed SW9: AS, Buttons_Switches_ThroughHole:SW_PUSH_6mm_h5mm, symbol Switch:SW_Push_45deg
- added J12: KEYBOARD, Pin_Headers:Pin_Header_Angled_1x06_Pitch1.27mm, symbol Connector_Generic:Conn_01x06
Connections:
- net +3V3: now also J12.6 (Pin_6)
- net CPU_NRST: now also J12.2 (Pin_2)
- net GND: now also J12.1 (Pin_1)
- net PA29_KEY_INT: now also J12.5 (Pin_5)
- net PA30_TWD0: now also J12.3 (Pin_3)
- net PA31_TWCK0: now also J12.4 (Pin_4)
- no-connect marks 69 -> 68
Other:
- moved on the sheet: R60, R61
